File: cad_files/color_sensor.kicad_pcb (KiCad board)
At the start: 2 copper layers, 49 x 77 mm, 75 parts, among them J1 USB_C_Receptacle_USB2.0, J2 RJ11, J3 RJ11, J4 PH, J5 PH, J6 Conn_02x03_Odd_Even, J7 Conn_01x05, J8 Conn_01x05, Q1 FDC304P, SW1 SW_Push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

Commit message: add pics
Routing:
- net /BACK_LIGHT: track 0.00 -> 18.4 mm, vias 0 -> 1
- net GND: track 45.8 -> 45.9 mm, vias 104 -> 112
Other:
- outline, holes or cut-outs redrawn
- net class Default removed
